Commit message: updated joint angles and robot position on table

File: ws4/src/msee22_description/urdf/msee22.urdf.xacro (robot description, xacro)
@@ -76,5 +76,5 @@
   <!-- if using jazzy, uncomment the lines 91-93 -->
    <xacro:ur_robot name="$(arg name)" tf_prefix="$(arg tf_prefix)" parent="table_top" joint_limits_parameters_file="$(arg joint_limit_params)" kinematics_parameters_file="$(arg kinematics_params)" physical_parameters_file="$(arg physical_params)" visual_parameters_file="$(arg visual_params)" safety_limits="$(arg safety_limits)" safety_pos_margin="$(arg safety_pos_margin)" safety_k_position="$(arg safety_k_position)">
-     <origin xyz="0 ${7.5*inch} ${1*inch}" rpy="0 0 ${-radians(135)}" />
+     <origin xyz="${-table_length/2 + 2.5*inch} ${-table_width/2 + 8*inch} 0" rpy="0 0 0" />
   </xacro:ur_robot>
   <!-- if using humble, uncomment the lines 97-136 -->
@@ -116,5 +116,5 @@
     trajectory_port="$(arg trajectory_port)"
   >
-  <origin xyz="0 ${7.5*inch} ${1*inch}" rpy="0 0 ${-radians(135)}" />
+    <origin xyz="${-table_length/2 + 2.5*inch} ${-table_width/2 + 8*inch} 0" rpy="0 0 0" />
   </xacro:ur_robot> -->
 </robot>

Commit message: corrected the screw axes and theta0

File: ws4/src/msee22_description/urdf/msee22.urdf.xacro (robot description, xacro)
@@ -76,5 +76,5 @@
   <!-- if using jazzy, uncomment the lines 91-93 -->
    <xacro:ur_robot name="$(arg name)" tf_prefix="$(arg tf_prefix)" parent="table_top" joint_limits_parameters_file="$(arg joint_limit_params)" kinematics_parameters_file="$(arg kinematics_params)" physical_parameters_file="$(arg physical_params)" visual_parameters_file="$(arg visual_params)" safety_limits="$(arg safety_limits)" safety_pos_margin="$(arg safety_pos_margin)" safety_k_position="$(arg safety_k_position)">
-     <origin xyz="${-table_length/2 + 2.5*inch} ${-table_width/2 + 8*inch} 0" rpy="0 0 0" />
+     <origin xyz="${-table_length/2 + 2.5*inch} ${-table_width/2 + 8*inch} 0" rpy="0 0 ${radians(180)}" />
   </xacro:ur_robot>
   <!-- if using humble, uncomment the lines 97-136 -->
@@ -116,5 +116,5 @@
     trajectory_port="$(arg trajectory_port)"
   >
-    <origin xyz="${-table_length/2 + 2.5*inch} ${-table_width/2 + 8*inch} 0" rpy="0 0 0" />
+    <origin xyz="${-table_length/2 + 2.5*inch} ${-table_width/2 + 8*inch} 0" rpy="0 0 ${radians(180)}" />
   </xacro:ur_robot> -->
 </robot>
